File: hardware/ethernet_rfid_reader.kicad_pcb (KiCad board)
At the start: 2 copper layers, 60 x 60 mm, 54 parts, among them J1 POWER, J2 ST-LINK, J3 UART, J4 RFID_RC522, J5 RJ45_Hanrun_HR911105A_Horizon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, U1 LM2596S-3.3, U2 STM32F103C8Tx, U3 ENC28J60x-SO, Y1 8M, Y2 25M

Commit message: Update hardware to v1.1
Parts:
- J2: footprint Connector_PinHeader_2.54mm:PinHeader_1x04_P2.54mm_Vertical -> Connector_PinHeader_2.54mm:PinHeader_1x06_P2.54mm_Vertical
- J4: footprint Libs:MODULE_CEG006900 -> libs:MODULE_CEG006900_1
- J5: footprint Libs:RJ45_Hanrun_HR911105A_Horizontal -> libs:RJ45_Hanrun_HR911105A_Horizontal
- S1, S2: footprint Libs:SW_TS-1187A-B-A-B -> libs:SW_TS-1187A-B-A-B
- moved L2 4.80 mm to (131.7, 118.2)
- moved R10 4.80 mm to (126.3, 118.4)
- moved C18 4.40 mm to (131.1, 120.4)
- moved R11 4.40 mm to (126.3, 120.4)
- moved C19 3.90 mm to (131.1, 124.9)
- moved R12 3.90 mm to (126.3, 124.9)
- moved R13 3.44 mm to (126.3, 126.9)
Connections:
- net /ETH_INT renamed /ETH_IRQ
- J2 pad 4: GND -> /SWOUT
- U2 pad 39: unconnected-(U2-PB3-Pad39) -> /SWOUT
Routing:
- net /NRST: track 42.7 -> 76.1 mm, vias 0 -> 1
- net /SWOUT: track 0.00 -> 25.2 mm, vias 0 -> 1
- net GND: track 204.9 -> 219.9 mm
- net /SWCLK: track 12.9 -> 18.7 mm
- net +3V3: track 248.6 -> 243.9 mm, vias 7 -> 8
- net /TPOUT+: track 46.8 -> 49.7 mm
- net /SWDIO: track 18.4 -> 15.7 mm, vias 0 -> 1
- net /TPOUT-: track 47.7 -> 50.4 mm
- net /TPIN-: track 57.1 -> 59.6 mm
- net /TPIN+: track 60.0 -> 62.4 mm
- net Net-(J5-TCT): track 19.6 -> 17.8 mm
- net Net-(J5-RCT): track 22.7 -> 23.9 mm
- added copper zone on F.Cu, net GND
Other:
- board text added: "3V3"
- board text added: ">"
- board text added: "Ethernet RFID Reader V1.1"
- board text added: "FAIL"
- board text added: "GND"
- board text added: "MISO"
- board text added: "MOSI"
- board text added: "NRST"
- board text added: "OK"
- board text added: "PWR"
- board text added: "RST"
- board text added: "RX"
- board text added: "SCK"
- board text added: "SDA"
- board text added: "SWC"
- board text added: "SWD"
- board text added: "SWO"
- board text added: "TX"
- board text added: "v"
