File: hardware/ethernet_rfid_reader.kicad_sch (KiCad schematic)
At the start: 54 parts, among them J1 POWER, J2 ST-LINK, J3 UART, J4 RFID_RC522, J5 RJ45_Hanrun_HR911105A_Horizon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, U1 LM2596S-3.3, U2 STM32F103C8Tx, U3 ENC28J60x-SO, Y1 8M, Y2 25M

Commit message: Update hardware to v1.1
Parts:
- J2: footprint Connector_PinHeader_2.54mm:PinHeader_1x04_P2.54mm_Vertical -> Connector_PinHeader_2.54mm:PinHeader_1x06_P2.54mm_Vertical; symbol Connector_Generic:Conn_01x04 -> Connector_Generic:Conn_01x06
- J4: footprint Libs:MODULE_CEG006900 -> libs:MODULE_CEG006900_1
- J5: footprint Libs:RJ45_Hanrun_HR911105A_Horizontal -> libs:RJ45_Hanrun_HR911105A_Horizontal
- S1, S2: footprint Libs:SW_TS-1187A-B-A-B -> libs:SW_TS-1187A-B-A-B
Connections:
- net GND: now also J2.6 (Pin_6); no longer J2.4 (Pin_4)
- net NRST: now also J2.5 (Pin_5)
- net SWOUT: now reaches U2.39 (PB3)
- net SWOUT: now also J2.4 (Pin_4)
- net ETH_INT renamed ETH_IRQ
- no-connect marks 22 -> 21
Changed lines of the file:
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@@
   (title_block
     (title "Ethernet RFID Reader ")
-    (date "2024-11-08")
-    (rev "1.0")
+    (date "2024-12-01")
+    (rev "1.1")
   )
   (junction (at 38.1 25.4) (diameter 0) (color 0 0 0 0)
@@
   (no_connect (at 144.78 78.74))
   (no_connect (at 144.78 93.98))
-  (no_connect (at 144.78 81.28))
   (no_connect (at 144.78 83.82))
   (no_connect (at 90.17 72.39))
@@
     (stroke (width 0) (type default))
   )
+  (wire (pts (xy 133.35 81.28) (xy 144.78 81.28))
+    (stroke (width 0) (type default))
+  )
   (wire (pts (xy 60.96 35.56) (xy 60.96 43.18))
     (stroke (width 0) (type default))
@@
     (stroke (width 0) (type default))
   )
-  (wire (pts (xy 26.67 62.23) (xy 26.67 64.77))
-    (stroke (width 0) (type default))
-  )
   (wire (pts (xy 260.35 57.15) (xy 269.24 57.15))
     (stroke (width 0) (type default))
@@
     (stroke (width 0) (type default))
   )
-  (wire (pts (xy 25.4 69.85) (xy 34.29 69.85))
-    (stroke (width 0) (type default))
-  )
   (wire (pts (xy 245.11 93.98) (xy 240.03 93.98))
     (stroke (width 0) (type default))
@@
     (stroke (width 0) (type default))
   )
-  (wire (pts (xy 26.67 73.66) (xy 26.67 72.39))
-    (stroke (width 0) (type default))
-  )
   (wire (pts (xy 177.8 55.88) (xy 186.69 55.88))
     (stroke (width 0) (type default))
@@
     (stroke (width 0) (type default))
   )
+  (wire (pts (xy 25.4 67.31) (xy 34.29 67.31))
+    (stroke (width 0) (type default))
+  )
   (wire (pts (xy 49.53 130.81) (xy 49.53 132.08))
     (stroke (width 0) (type default))
@@
     (stroke (width 0) (type default))
   )
+  (wire (pts (xy 25.4 77.47) (xy 26.67 77.47))
+    (stroke (width 0) (type default))
+  )
   (wire (pts (xy 60.96 64.77) (xy 59.69 64.77))
     (stroke (width 0) (type default))
   )
+  (wire (pts (xy 25.4 74.93) (xy 34.29 74.93))
+    (stroke (width 0) (type default))
+  )
   (wire (pts (xy 212.09 59.69) (xy 224.79 59.69))
     (stroke (width 0) (type default))
@@
     (stroke (width 0) (type default))
   )
-  (wire (pts (xy 26.67 72.39) (xy 25.4 72.39))
-    (stroke (width 0) (type default))
-  )
   (wire (pts (xy 100.33 160.02) (xy 100.33 158.75))
     (stroke (width 0) (type default))
@@
     (stroke (width 0) (type default))
   )
-  (wire (pts (xy 26.67 64.77) (xy 25.4 64.77))
-    (stroke (width 0) (type default))
-  )
   (wire (pts (xy 140.97 25.4) (xy 140.97 24.13))
     (stroke (width 0) (type default))
@@
     (stroke (width 0) (type default))
   )
+  (wire (pts (xy 26.67 62.23) (xy 26.67 64.77))
+    (stroke (width 0) (type default))
+  )
   (wire (pts (xy 74.93 39.37) (xy 74.93 43.18))
     (stroke (width 0) (type default))
@@
     (stroke (width 0) (type default))
   )
-  (wire (pts (xy 25.4 67.31) (xy 34.29 67.31))
+  (wire (pts (xy 25.4 69.85) (xy 34.29 69.85))
     (stroke (width 0) (type default))
   )
@@
     (stroke (width 0) (type default))
   )
+  (wire (pts (xy 25.4 72.39) (xy 34.29 72.39))
+    (stroke (width 0) (type default))
+  )
   (wire (pts (xy 245.11 92.71) (xy 245.11 93.98))
     (stroke (width 0) (type default))
@@
     (stroke (width 0) (type default))
   )
+  (wire (pts (xy 25.4 64.77) (xy 26.67 64.77))
+    (stroke (width 0) (type default))
+  )
   (wire (pts (xy 165.1 39.37) (xy 167.64 39.37))
     (stroke (width 0) (type default))
@@
     (stroke (width 0) (type default))
   )
+  (wire (pts (xy 26.67 77.47) (xy 26.67 78.74))
+    (stroke (width 0) (type default))
+  )
   (wire (pts (xy 133.35 50.8) (xy 144.78 50.8))
     (stroke (width 0) (type default))
@@
     (effects (font (size 1.27 1.27)) (justify left bottom))
   )
+  (label "SWOUT" (at 29.21 72.39 0) (fields_autoplaced)
+    (effects (font (size 1.27 1.27)) (justify left bottom))
+  )
   (label "READ_FAIL" (at 134.62 76.2 0) (fields_autoplaced)
     (effects (font (size 1.27 1.27)) (justify left bottom))
@@
     (effects (font (size 1.27 1.27)) (justify left bottom))
   )
+  (label "NRST" (at 29.21 74.93 0) (fields_autoplaced)
+    (effects (font (size 1.27 1.27)) (justify left bottom))
+  )
   (label "ETH_OSC2" (at 213.36 80.01 0) (fields_autoplaced)
     (effects (font (size 1.27 1.27)) (justify left bottom))
@@
     (effects (font (size 1.27 1.27)) (justify left bottom))
   )
-  (label "ETH_INT" (at 213.36 64.77 0) (fields_autoplaced)
+  (label "ETH_IRQ" (at 213.36 64.77 0) (fields_autoplaced)
     (effects (font (size 1.27 1.27)) (justify left bottom))
   )
@@
     (effects (font (size 1.27 1.27)) (justify left bottom))
   )
-  (label "ETH_INT" (at 190.5 66.04 0) (fields_autoplaced)
+  (label "ETH_IRQ" (at 190.5 66.04 0) (fields_autoplaced)
     (effects (font (size 1.27 1.27)) (justify left bottom))
   )
@@
     (effects (font (size 1.27 1.27)) (justify left bottom))
   )
+  (label "SWOUT" (at 134.62 81.28 0) (fields_autoplaced)
+    (effects (font (size 1.27 1.27)) (justify left bottom))
+  )
   (label "HSE_IN" (at 134.62 55.88 0) (fields_autoplaced)
     (effects (font (size 1.27 1.27)) (justify left bottom))
@@
     )
   )
-  (symbol (lib_id "power:GND") (at 26.67 73.66 0) (unit 1)
+  (symbol (lib_id "power:GND") (at 26.67 78.74 0) (unit 1)
     (in_bom yes) (on_board yes) (dnp no) (fields_autoplaced)
-    (property "Reference" "#PWR012" (at 26.67 80.01 0)
+    (property "Reference" "#PWR012" (at 26.67 85.09 0)
       (effects (font (size 1.27 1.27)) hide)
     )
-    (property "Value" "GND" (at 26.67 78.74 0)
+    (property "Value" "GND" (at 26.67 83.82 0)
       (effects (font (size 1.27 1.27)))
     )
-    (property "Footprint" "" (at 26.67 73.66 0)
+    (property "Footprint" "" (at 26.67 78.74 0)
       (effects (font (size 1.27 1.27)) hide)
     )
-    (property "Datasheet" "" (at 26.67 73.66 0)
+    (property "Datasheet" "" (at 26.67 78.74 0)
       (effects (font (size 1.27 1.27)) hide)
     )
@@
   )
   (symbol (lib_id "power:+3V3") (at 210.82 72.39 90) (unit 1)
-    (in_bom yes) (on_board yes) (dnp no) (fields_autoplaced)
+    (in_bom yes) (on_board yes) (dnp no)
     (property "Reference" "#PWR026" (at 214.63 72.39 0)
       (effects (font (size 1.27 1.27)) hide)
@@
       (effects (font (size 1.27 1.27)) (justify right))
     )
-    (property "Footprint" "Libs:SW_TS-1187A-B-A-B" (at 49.53 102.87 0)
+    (property "Footprint" "libs:SW_TS-1187A-B-A-B" (at 49.53 102.87 0)
       (effects (font (size 1.27 1.27)) (justify bottom) hide)
     )
@@
       (effects (font (size 1.27 1.27)))
     )
-    (property "Footprint" "Libs:MODULE_CEG006900" (at 85.09 72.39 0)
+    (property "Footprint" "libs:MODULE_CEG006900_1" (at 85.09 72.39 0)
       (effects (font (size 1.27 1.27)) hide)
     )
@@
     )
   )
-  (symbol (lib_id "Connector_Generic:Conn_01x04") (at 20.32 67.31 0) (mirror y) (unit 1)
+  (symbol (lib_id "Connector_Generic:Conn_01x06") (at 20.32 69.85 0) (mirror y) (unit 1)
     (in_bom yes) (on_board yes) (dnp no)
-    (property "Reference" "J2" (at 16.51 58.42 0)
+    (property "Reference" "J2" (at 16.51 60.96 0)
       (effects (font (size 1.27 1.27)))
     )
-    (property "Value" "ST-LINK" (at 17.78 60.96 0)
+    (property "Value" "ST-LINK" (at 17.78 63.5 0)
       (effects (font (size 1.27 1.27)))
     )
-    (property "Footprint" "Connector_PinHeader_2.54mm:PinHeader_1x04_P2.54mm_Vertical" (at 20.32 67.31 0)
+    (property "Footprint" "Connector_PinHeader_2.54mm:PinHeader_1x06_P2.54mm_Vertical" (at 20.32 69.85 0)
       (effects (font (size 1.27 1.27)) hide)
     )
-    (property "Datasheet" "~" (at 20.32 67.31 0)
+    (property "Datasheet" "~" (at 20.32 69.85 0)
       (effects (font (size 1.27 1.27)) hide)
     )
@@
     (pin "1")
     (pin "3")
+    (pin "6")
+    (pin "5")
     (instances
       (project "ethernet_rfid_reader"
@@
       (effects (font (size 1.27 1.27)) (justify right))
     )
-    (property "Footprint" "Libs:SW_TS-1187A-B-A-B" (at 21.59 120.65 0)
+    (property "Footprint" "libs:SW_TS-1187A-B-A-B" (at 21.59 120.65 0)
       (effects (font (size 1.27 1.27)) (justify bottom) hide)
     )
@@
       (effects (font (size 1.27 1.27)))
     )
-    (property "Footprint" "Libs:RJ45_Hanrun_HR911105A_Horizontal" (at 74.93 151.13 0)
+    (property "Footprint" "libs:RJ45_Hanrun_HR911105A_Horizontal" (at 74.93 151.13 0)
       (effects (font (size 1.27 1.27)) hide)
     )
